File: stickcontroller/stickcontroller.kicad_pcb (KiCad board)
At the start: 2 copper layers, 7.5 x 2 mm, 20 parts, among them J1 USB_B_Micro, J2 Conn_01x04, J3 Conn_01x02, J4 Conn_02x03_Odd_Even, SW1 SW_Push, SW2 SW_Push, SW3 SW_Push, SW4 SW_Push, SW5 SW_Push, SW6 SW_Push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

Commit message: Add files via upload
Parts:
- removed J1: USB_B_Micro, Connector_USB:USB_Micro-AB_Molex_47590-0001
- removed J2: Conn_01x04, Connector_PinHeader_2.54mm:PinHeader_1x04_P2.54mm_Vertical
- removed J3: Conn_01x02, Connector_PinHeader_2.54mm:PinHeader_1x02_P2.54mm_Vertical
- removed SW4, SW5, SW6, SW7: SW_Push, Button_Switch_SMD:Panasonic_EVQPUM_EVQPUD
- added B1: 4-direction-joystick, Button_Switch_THT:JS5208, F.Cu at (176.4, 84.9)
- added C4: 0.1uF, Capacitor_SMD:C_0805_2012Metric_Pad1.15x1.40mm_HandSolder, B.Cu at (182.9, 105.6)
- added C5: 10uF, Capacitor_SMD:C_0805_2012Metric_Pad1.15x1.40mm_HandSolder, B.Cu at (180.9, 105.6)
- added D+ D-: Conn_01x02, Connector_PinHeader_2.54mm:PinHeader_1x02_P2.54mm_Vertical, B.Cu at (185.6, 98.2)
- added PPT: SW_Push, Button_Switch_SMD:Reichelt_RAFI_Kurzhubtaster, F.Cu at (182.7, 106.1)
- added PPT: Conn_01x02, Connector_PinHeader_2.54mm:PinHeader_1x02_P2.54mm_Vertical, B.Cu at (173.8, 103.6)
- added RST: Jumper_NO_Small, Jumper:SolderJumper-2_P1.3mm_Open_Pad1.0x1.5mm, B.Cu at (182.9, 101.7)
- C1, C2, C3, D1, R1, R2, R3, U1: moved to B.Cu
- J4: value Conn_02x03_Odd_Even -> Conn_02x03; moved to B.Cu
- SW1: footprint Button_Switch_SMD:Panasonic_EVQPUM_EVQPUD -> Button_Switch_SMD:Reichelt_RAFI_Kurzhubtaster
- SW2, SW3: footprint Button_Switch_SMD:Panasonic_EVQPUM_EVQPUD -> Button_Switch_SMD:Reichelt_RAFI_Kurzhubtaster; moved to F.Cu
- Y1: value Crystal -> 16MHz; footprint Crystal:Crystal_SMD_TXC_7A-2Pin_5x3.2mm -> Crystal:Crystal_SMD_5032-2Pin_5.0x3.2mm_HandSoldering; moved to B.Cu
- moved SW3 80.2 mm to (194.5, 97.8), turned to 90 degrees
- moved R1 68.4 mm to (188.6, 74.5), turned to 0 degrees
- moved SW2 67.4 mm to (186.4, 83.7)
- moved D1 67.1 mm to (188.6, 72.4), turned to 180 degrees
- moved R2 60.7 mm to (189.3, 96.5), turned to 180 degrees
- moved J4 59.2 mm to (186.2, 105.9)
- moved C2 58.6 mm to (176.4, 72.8), turned to 180 degrees
- moved C3 58.2 mm to (189.3, 94.5), turned to 180 degrees
- moved R3 57.8 mm to (189.3, 98.4), turned to 180 degrees
- moved C1 55.7 mm to (181.9, 72.8), turned to 0 degrees
- moved Y1 54.9 mm to (179.2, 75.9)
- moved U1 53.6 mm to (190.9, 86.7), turned to 90 degrees
- moved SW1 51.2 mm to (174.3, 75.7), turned to 0 degrees
Connections:
- SW1 pad 1: GND -> Net-(SW1-Pad1)
- SW1 pad 2: Net-(J4-Pad5) -> GND
- U1 pad 18: Net-(SW2-Pad1) -> Net-(B1-Pad3)
- U1 pad 19: Net-(SW3-Pad1) -> Net-(B1-Pad2)
- U1 pad 25: Net-(SW6-Pad1) -> Net-(SW1-Pad1)
- U1 pad 26: Net-(U1-Pad26) -> Net-(SW2-Pad1)
- U1 pad 27: Net-(U1-Pad27) -> Net-(SW3-Pad1)
Routing:
- net GND: track 2.75 -> 41.3 mm, vias 0 -> 2
- net Net-(SW2-Pad1): track 40.9 -> 12.1 mm
- net Net-(J4-Pad4): track 0.00 -> 27.1 mm
- net Net-(R3-Pad1): track 30.7 -> 7.59 mm
- net Net-(SW6-Pad1): track 22.8 -> 0.00 mm, vias 1 -> 0
- net Net-(J4-Pad1): track 0.00 -> 22.6 mm
- net Net-(SW1-Pad1): track 0.00 -> 21.5 mm, vias 0 -> 1
- net +5V: track 57.5 -> 77.0 mm, vias 0 -> 3
- net Net-(J4-Pad3): track 0.00 -> 19.3 mm
- net Net-(C1-Pad1): track 9.56 -> 28.6 mm
- net Net-(R2-Pad1): track 23.0 -> 5.30 mm
- net Net-(B1-Pad3): track 0.00 -> 17.5 mm, vias 0 -> 1
- net Net-(SW3-Pad1): track 33.9 -> 16.4 mm
- net Net-(B1-Pad2): track 0.00 -> 16.4 mm, vias 0 -> 1
- net Net-(C2-Pad1): track 9.31 -> 25.3 mm
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- added copper zone on B.Cu, net GND
- added copper zone on F.Cu, net GND
Other:
- board size 7.5 x 2 mm -> 32.8 x 42.7 mm
- net class +5V added: clearance 0.4, trace_width 0.5, via_dia 0.8, via_drill 0.4

Commit message: Add files via upload
Parts:
- added Uin: Conn_01x02, Connector_PinHeader_2.54mm:PinHeader_1x02_P2.54mm_Vertical, B.Cu at (171.3, 93.5)
- renumbered PPT to SWPPT1
Routing:
- net +5V: track 77.0 -> 91.8 mm
- net GND: track 41.3 -> 40.5 mm
Changed lines of the file:
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@@
     (thickness 1.6)
     (drawings 107)
-    (tracks 196)
+    (tracks 200)
     (zones 0)
-    (modules 20)
+    (modules 21)
     (nets 41)
   )
@@
     (39 F.Mask user)
     (40 Dwgs.User user)
-    (41 Cmts.User user)
-    (42 Eco1.User user)
+    (41 Cmts.User user hide)
+    (42 Eco1.User user hide)
     (43 Eco2.User user)
     (44 Edge.Cuts user)
@@
   )
   (setup
-    (last_trace_width 0.4)
+    (last_trace_width 0.5)
     (user_trace_width 0.4)
     (user_trace_width 0.5)
@@
   )
   (module Connector_PinHeader_2.54mm:PinHeader_1x02_P2.54mm_Vertical (layer B.Cu)
+    (at 171.33 93.48 270)
+    (descr "Through hole straight pin header, 1x02, 2.54mm pitch, single row")
+    (tags "Through hole pin header THT 1x02 2.54mm single row")
+    (fp_text reference Uin (at 0 2.33 270) (layer B.SilkS)
+      (effects (font (size 1 1) (thickness 0.15)) (justify mirror))
+    )
+    (fp_text value Conn_01x02 (at 0 -4.87 270) (layer B.Fab)
+      (effects (font (size 1 1) (thickness 0.15)) (justify mirror))
+    )
+    (fp_text user %R (at 0 -1.27) (layer B.Fab)
+      (effects (font (size 1 1) (thickness 0.15)) (justify mirror))
+    )
+    (fp_line (start 1.8 1.8) (end -1.8 1.8) (layer B.CrtYd) (width 0.05))
+    (fp_line (start 1.8 -4.35) (end 1.8 1.8) (layer B.CrtYd) (width 0.05))
+    (fp_line (start -1.8 -4.35) (end 1.8 -4.35) (layer B.CrtYd) (width 0.05))
+    (fp_line (start -1.8 1.8) (end -1.8 -4.35) (layer B.CrtYd) (width 0.05))
+    (fp_line (start -1.33 1.33) (end 0 1.33) (layer B.SilkS) (width 0.12))
+    (fp_line (start -1.33 0) (end -1.33 1.33) (layer B.SilkS) (width 0.12))
+    (fp_line (start -1.33 -1.27) (end 1.33 -1.27) (layer B.SilkS) (width 0.12))
+    (fp_line (start 1.33 -1.27) (end 1.33 -3.87) (layer B.SilkS) (width 0.12))
+    (fp_line (start -1.33 -1.27) (end -1.33 -3.87) (layer B.SilkS) (width 0.12))
+    (fp_line (start -1.33 -3.87) (end 1.33 -3.87) (layer B.SilkS) (width 0.12))
+    (fp_line (start -1.27 0.635) (end -0.635 1.27) (layer B.Fab) (width 0.1))
+    (fp_line (start -1.27 -3.81) (end -1.27 0.635) (layer B.Fab) (width 0.1))
+    (fp_line (start 1.27 -3.81) (end -1.27 -3.81) (layer B.Fab) (width 0.1))
+    (fp_line (start 1.27 1.27) (end 1.27 -3.81) (layer B.Fab) (width 0.1))
+    (fp_line (start -0.635 1.27) (end 1.27 1.27) (layer B.Fab) (width 0.1))
+    (pad 2 thru_hole oval (at 0 -2.54 270) (size 1.7 1.7) (drill 1) (layers *.Cu *.Mask)
+      (net 10 +5V))
+    (pad 1 thru_hole rect (at 0 0 270) (size 1.7 1.7) (drill 1) (layers *.Cu *.Mask)
+      (net 1 GND))
+    (model ${KISYS3DMOD}/Connector_PinHeader_2.54mm.3dshapes/PinHeader_1x02_P2.54mm_Vertical.wrl
+      (at (xyz 0 0 0))
+      (scale (xyz 1 1 1))
+      (rotate (xyz 0 0 0))
+    )
+  )
+  (module Connector_PinHeader_2.54mm:PinHeader_1x02_P2.54mm_Vertical (layer B.Cu)
     (at 185.64 98.16)
     (descr "Through hole straight pin header, 1x02, 2.54mm pitch, single row")
@@
   (module Button_Switch_SMD:Reichelt_RAFI_Kurzhubtaster (layer F.Cu)
     (at 182.7 106.1 90)
-    (fp_text reference PPT (at -1.86 -0.3 180) (layer F.SilkS)
+    (fp_text reference SWPPT1 (at -1.86 -0.3 180) (layer F.SilkS)
       (effects (font (size 1 1) (thickness 0.15)))
     )
@@
   (gr_line (start 197.96679 72.00584) (end 197.53448 70.98552) (layer Edge.Cuts) (width 0.0254))
   (gr_line (start 199.06712 86.7767) (end 199.1705 85.3952) (layer Edge.Cuts) (width 0.0254))
-  (segment (start 180.92 104.595) (end 180.92 101.71) (width 0.5) (layer B.Cu) (net 1))
-  (segment (start 180.92 101.71) (end 180.92 101.71) (width 0.25) (layer B.Cu) (net 1))
-  (via (at 180.92 101.71) (size 1.6) (drill 0.8) (layers F.Cu B.Cu) (net 1))
   (segment (start 187.890001 101.669999) (end 188.74 100.82) (width 0.4) (layer B.Cu) (net 1))
   (segment (start 187.489999 102.070001) (end 187.890001 101.669999) (width 0.4) (layer B.Cu) (net 1))
@@
   (segment (start 185.2 88.3) (end 179.68 88.3) (width 0.4) (layer B.Cu) (net 1))
   (via (at 191.7 94.40501) (size 0.8) (drill 0.4) (layers F.Cu B.Cu) (net 1))
+  (segment (start 180.92 103.28) (end 180.92 104.595) (width 0.5) (layer B.Cu) (net 1))
+  (via (at 180.53 102.56) (size 1.6) (drill 0.8) (layers F.Cu B.Cu) (net 1))
+  (segment (start 180.53 102.56) (end 180.92 103.28) (width 0.5) (layer B.Cu) (net 1))
   (segment (start 185.2 85.9) (end 179.9 85.9) (width 0.25) (layer B.Cu) (net 2))
   (segment (start 179.9 85.9) (end 179.9 85.9) (width 0.25) (layer B.Cu) (net 2))
@@
   (segment (start 192.378625 90.33) (end 191.5 90.33) (width 0.5) (layer F.Cu) (net 10))
   (segment (start 196.625001 94.576376) (end 192.378625 90.33) (width 0.5) (layer F.Cu) (net 10))
+  (segment (start 184.186814 89.1) (end 185.2 89.1) (width 0.5) (layer B.Cu) (net 10))
+  (segment (start 182.678407 90.608407) (end 184.186814 89.1) (width 0.5) (layer B.Cu) (net 10))
+  (segment (start 173.87 93.48) (end 182.678407 93.48) (width 0.5) (layer B.Cu) (net 10))
+  (segment (start 182.678407 93.48) (end 182.678407 90.608407) (width 0.5) (layer B.Cu) (net 10))
   (segment (start 187.525 72.39) (end 187.525 74.51) (width 0.25) (layer B.Cu) (net 11))
   (segment (start 188.025 98.16) (end 188.295 98.43) (width 0.25) (layer B.Cu) (net 12))
@@
   (segment (start 181.824999 97.695999) (end 181.824999 103.060001) (width 0.25) (layer B.Cu) (net 18))
   (segment (start 188.5 92.4) (end 188.5 93.4) (width 0.25) (layer B.Cu) (net 18))
-  (segment (start 179.89499 98.88001) (end 186.375 92.4) (width 0.25) (layer B.Cu) (net 19))
   (segment (start 186.375 92.4) (end 186.9 92.4) (width 0.25) (layer B.Cu) (net 19))
-  (segment (start 179.89499 105.15818) (end 179.89499 98.88001) (width 0.25) (layer B.Cu) (net 19))
-  (segment (start 180.23682 105.50001) (end 179.89499 105.15818) (width 0.25) (layer B.Cu) (net 19))
+  (segment (start 186.2 105.9) (end 185.1 105.9) (width 0.25) (layer B.Cu) (net 19))
+  (segment (start 185.1 105.9) (end 184.70001 105.50001) (width 0.25) (layer B.Cu) (net 19))
   (segment (start 184.70001 105.50001) (end 180.23682 105.50001) (width 0.25) (layer B.Cu) (net 19))
-  (segment (start 185.1 105.9) (end 184.70001 105.50001) (width 0.25) (layer B.Cu) (net 19))
-  (segment (start 186.2 105.9) (end 185.1 105.9) (width 0.25) (layer B.Cu) (net 19))
+  (segment (start 179.404999 99.370001) (end 186.375 92.4) (width 0.25) (layer B.Cu) (net 19))
+  (segment (start 179.404999 104.668189) (end 179.404999 99.370001) (width 0.25) (layer B.Cu) (net 19))
+  (segment (start 180.23682 105.50001) (end 179.404999 104.668189) (width 0.25) (layer B.Cu) (net 19))
   (segment (start 192.5 93.4) (end 192.5 92.4) (width 0.25) (layer B.Cu) (net 20))
   (segment (start 192.5 94.89) (end 192.5 93.4) (width 0.25) (layer B.Cu) (net 20))

Commit message: Add files via upload
Parts:
- added D2: LED, LED_SMD:LED_0805_2012Metric_Pad1.15x1.40mm_HandSolder, B.Cu at (188.6, 70.3)
- added R4: 1K, Resistor_SMD:R_0805_2012Metric_Pad1.15x1.40mm_HandSolder, B.Cu at (188.6, 68.3)
- turned D1 to 0 degrees
Routing:
- net Net-(R4-Pad2): track 0.00 -> 33.4 mm, vias 0 -> 2
- net Net-(SW2-Pad1): track 12.1 -> 4.36 mm
- net GND: track 40.5 -> 43.4 mm, vias 2 -> 3
- net +5V: track 91.8 -> 94.3 mm
- net Net-(D2-Pad2): track 0.00 -> 2.01 mm
- net Net-(D1-Pad2): track 2.12 -> 2.97 mm
Other:
- board text added: "+5V"
- board text added: "GND"
- board text added: "Kaiser J. FSG Heinkel 2020 V1.0"

Commit message: Add files via upload
Parts:
- added F1: 500mA, Fuse:Fuse_0603_1608Metric, B.Cu at (178.9, 93.5)
Connections:
- Uin pad 2: +5V -> Net-(F1-Pad2)
Routing:
- net GND: track 43.4 -> 62.9 mm
- net +5V: track 94.3 -> 88.5 mm
- net Net-(F1-Pad2): track 0.00 -> 4.24 mm
Changed lines of the file:
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@@
     (thickness 1.6)
     (drawings 110)
-    (tracks 223)
+    (tracks 229)
     (zones 0)
-    (modules 23)
-    (nets 42)
+    (modules 24)
+    (nets 43)
   )
   (page A4)
@@
   )
   (setup
-    (last_trace_width 0.25)
+    (last_trace_width 0.5)
     (user_trace_width 0.4)
     (user_trace_width 0.5)
@@
   (net 40 "Net-(D2-Pad2)")
   (net 41 "Net-(R4-Pad2)")
+  (net 42 "Net-(F1-Pad2)")
   (net_class Default "Dies ist die voreingestellte Netzklasse."
     (clearance 0.2)
@@
     (add_net "Net-(D1-Pad2)")
     (add_net "Net-(D2-Pad2)")
+    (add_net "Net-(F1-Pad2)")
     (add_net "Net-(J3-Pad1)")
     (add_net "Net-(J3-Pad2)")
@@
     (uvia_drill 0.1)
   )
+  (module Fuse:Fuse_0603_1608Metric (layer B.Cu)
+    (at 178.9 93.48 180)
+    (descr "Fuse SMD 0603 (1608 Metric), square (rectangular) end terminal, IPC_7351 nominal, (Body size source: http://www.tortai-tech.com/upload/download/2011102023233369053.pdf), generated with kicad-footprint-generator")
+    (tags resistor)
+    (attr smd)
+    (fp_text reference F1 (at 0 1.43) (layer B.SilkS)
+      (effects (font (size 1 1) (thickness 0.15)) (justify mirror))
+    )
+    (fp_text value 500mA (at 0 -1.43) (layer B.Fab)
+      (effects (font (size 1 1) (thickness 0.15)) (justify mirror))
+    )
+    (fp_text user %R (at 0 0) (layer B.Fab)
+      (effects (font (size 0.4 0.4) (thickness 0.06)) (justify mirror))
+    )
+    (fp_line (start 1.48 -0.73) (end -1.48 -0.73) (layer B.CrtYd) (width 0.05))
+    (fp_line (start 1.48 0.73) (end 1.48 -0.73) (layer B.CrtYd) (width 0.05))
+    (fp_line (start -1.48 0.73) (end 1.48 0.73) (layer B.CrtYd) (width 0.05))
+    (fp_line (start -1.48 -0.73) (end -1.48 0.73) (layer B.CrtYd) (width 0.05))
+    (fp_line (start -0.162779 -0.51) (end 0.162779 -0.51) (layer B.SilkS) (width 0.12))
+    (fp_line (start -0.162779 0.51) (end 0.162779 0.51) (layer B.SilkS) (width 0.12))
+    (fp_line (start 0.8 -0.4) (end -0.8 -0.4) (layer B.Fab) (width 0.1))
+    (fp_line (start 0.8 0.4) (end 0.8 -0.4) (layer B.Fab) (width 0.1))
+    (fp_line (start -0.8 0.4) (end 0.8 0.4) (layer B.Fab) (width 0.1))
+    (fp_line (start -0.8 -0.4) (end -0.8 0.4) (layer B.Fab) (width 0.1))
+    (pad 2 smd roundrect (at 0.7875 0 180) (size 0.875 0.95) (layers B.Cu B.Paste B.Mask) (roundrect_rratio 0.25)
+      (net 42 "Net-(F1-Pad2)"))
+    (pad 1 smd roundrect (at -0.7875 0 180) (size 0.875 0.95) (layers B.Cu B.Paste B.Mask) (roundrect_rratio 0.25)
+      (net 10 +5V))
+    (model ${KISYS3DMOD}/Fuse.3dshapes/Fuse_0603_1608Metric.wrl
+      (at (xyz 0 0 0))
+      (scale (xyz 1 1 1))
+      (rotate (xyz 0 0 0))
+    )
+  )
   (module Resistor_SMD:R_0805_2012Metric_Pad1.15x1.40mm_HandSolder (layer B.Cu)
     (at 188.6 68.28)
@@
     (fp_line (start -0.635 1.27) (end 1.27 1.27) (layer B.Fab) (width 0.1))
     (pad 2 thru_hole oval (at 0 -2.54 270) (size 1.7 1.7) (drill 1) (layers *.Cu *.Mask)
-      (net 10 +5V))
+      (net 42 "Net-(F1-Pad2)"))
     (pad 1 thru_hole rect (at 0 0 270) (size 1.7 1.7) (drill 1) (layers *.Cu *.Mask)
       (net 1 GND))
@@
   (segment (start 196.6 89.9) (end 197.545002 89.9) (width 0.4) (layer B.Cu) (net 1))
   (segment (start 197.545002 89.9) (end 197.75003 89.694971) (width 0.4) (layer B.Cu) (net 1))
-  (segment (start 185.2 88.3) (end 179.68 88.3) (width 0.4) (layer B.Cu) (net 1))
   (via (at 191.7 94.40501) (size 0.8) (drill 0.4) (layers F.Cu B.Cu) (net 1))
   (segment (start 180.92 103.28) (end 180.92 104.595) (width 0.5) (layer B.Cu) (net 1))
@@
   (segment (start 189.615 70.29) (end 189.615 70.3) (width 0.5) (layer B.Cu) (net 1))
   (via (at 194.06 76.46) (size 1.6) (drill 0.8) (layers F.Cu B.Cu) (net 1))
+  (segment (start 184.36 88.3) (end 185.2 88.3) (width 0.5) (layer B.Cu) (net 1))
+  (segment (start 174.81 72.78) (end 173.449979 74.140021) (width 0.5) (layer B.Cu) (net 1))
+  (segment (start 173.449979 74.140021) (end 173.449979 82.363165) (width 0.5) (layer B.Cu) (net 1))
+  (segment (start 179.386814 88.3) (end 184.36 88.3) (width 0.5) (layer B.Cu) (net 1))
+  (segment (start 175.385 72.78) (end 174.81 72.78) (width 0.5) (layer B.Cu) (net 1))
+  (segment (start 173.449979 82.363165) (end 179.386814 88.3) (width 0.5) (layer B.Cu) (net 1))
   (segment (start 185.2 85.9) (end 179.9 85.9) (width 0.25) (layer B.Cu) (net 2))
   (segment (start 179.9 85.9) (end 179.9 85.9) (width 0.25) (layer B.Cu) (net 2))
@@
   (segment (start 192.378625 90.33) (end 191.5 90.33) (width 0.5) (layer F.Cu) (net 10))
   (segment (start 196.625001 94.576376) (end 192.378625 90.33) (width 0.5) (layer F.Cu) (net 10))
-  (segment (start 184.186814 89.1) (end 185.2 89.1) (width 0.5) (layer B.Cu) (net 10))
-  (segment (start 182.678407 90.608407) (end 184.186814 89.1) (width 0.5) (layer B.Cu) (net 10))
-  (segment (start 173.87 93.48) (end 182.678407 93.48) (width 0.5) (layer B.Cu) (net 10))
-  (segment (start 182.678407 93.48) (end 182.678407 90.608407) (width 0.5) (layer B.Cu) (net 10))
   (segment (start 194.1 90.82) (end 194.1 91.15) (width 0.5) (layer B.Cu) (net 10))
   (segment (start 194.1 91.15) (end 194.1 92.4) (width 0.5) (layer B.Cu) (net 10))
@@
   (segment (start 194.211836 78.476834) (end 196.6 80.864998) (width 0.5) (layer B.Cu) (net 10))
   (segment (start 190.276834 78.476834) (end 194.211836 78.476834) (width 0.5) (layer B.Cu) (net 10))
+  (segment (start 179.6875 93.48) (end 182.678407 93.48) (width 0.5) (layer B.Cu) (net 10))
+  (segment (start 184.186814 89.1) (end 185.2 89.1) (width 0.5) (layer B.Cu) (net 10))
+  (segment (start 182.678407 90.608407) (end 184.186814 89.1) (width 0.5) (layer B.Cu) (net 10))
+  (segment (start 182.678407 93.48) (end 182.678407 90.608407) (width 0.5) (layer B.Cu) (net 10))
   (segment (start 187.525 74.44) (end 189.575 72.39) (width 0.25) (layer B.Cu) (net 11))
   (segment (start 187.525 74.51) (end 187.525 74.44) (width 0.25) (layer B.Cu) (net 11))
@@
   (segment (start 191.56 68.28) (end 191.59 68.31) (width 0.25) (layer B.Cu) (net 41))
   (segment (start 189.625 68.28) (end 191.56 68.28) (width 0.25) (layer B.Cu) (net 41))
+  (segment (start 178.1125 93.48) (end 173.87 93.48) (width 0.5) (layer B.Cu) (net 42))
   (zone (net 1) (net_name GND) (layer B.Cu) (hatch edge 0.508)
     (connect_pads (clearance 0.508))

Commit message: Add files via upload
Parts:
- removed the Uin at (171.3, 93.5)
- added SF: Conn_01x02, Connector_Wire:SolderWirePadOval_2, B.Cu at (174.5, 103.9)
- added Uin: Conn_01x02, Connector_Wire:SolderWirePadOval_2, B.Cu at (171.0, 93.7)
- D+ D-: footprint Connector_PinHeader_2.54mm:PinHeader_1x02_P2.54mm_Vertical -> Connector_Wire:SolderWirePadOval_2
- PPT: footprint Connector_PinHeader_2.54mm:PinHeader_1x02_P2.54mm_Vertical -> Connector_Wire:SolderWirePadOval_2
- moved PPT 3.06 mm to (172.5, 100.8), turned to 90 degrees
- moved D+ D- 0.28 mm to (185.9, 98.3), turned to 180 degrees
Routing:
- net GND: track 62.9 -> 88.1 mm
- net Net-(J5-Pad1): track 0.00 -> 18.5 mm, vias 0 -> 1
- net Net-(J3-Pad1): track 21.2 -> 25.1 mm
- net Net-(J3-Pad2): track 16.3 -> 12.3 mm
- net Net-(F1-Pad2): track 4.24 -> 5.19 mm
- net /D+: track 3.01 -> 2.49 mm
Other:
- board text added: "500mA"
