File: stickcontroller/stickcontroller.sch (KiCad schematic (older format))
At the start: 19 parts, among them J1 USB_B_Micro, J2 Conn_01x04, J3 Conn_01x02, J4 Conn_02x03_Odd_Even, SW1 SW_Push, SW2 SW_Push, SW3 SW_Push, U1 ATmega32U4-AU, Y1 Crystal

Commit message: Add files via upload
Parts:
- removed J1: USB_B_Micro, Connector_USB:USB_Micro-AB_Molex_47590-0001, symbol Connector:USB_B_Micro
- removed J2: Conn_01x04, Connector_PinHeader_2.54mm:PinHeader_1x04_P2.54mm_Vertical, symbol Connector_Generic:Conn_01x04
- removed SWReset1: SW_Push, Button_Switch_SMD:Panasonic_EVQPUM_EVQPUD, symbol Switch:SW_Push
- added C4: 0.1uF, Capacitor_SMD:C_0805_2012Metric_Pad1.15x1.40mm_HandSolder, symbol Device:C
- added C5: 10uF, Capacitor_SMD:C_0805_2012Metric_Pad1.15x1.40mm_HandSolder, symbol Device:C
- added J1: Conn_01x02, Connector_PinHeader_2.54mm:PinHeader_1x02_P2.54mm_Vertical, symbol Connector_Generic:Conn_01x02
- added JP1: Jumper_NO_Small, Jumper:SolderJumper-2_P1.3mm_Open_Pad1.0x1.5mm, symbol Device:Jumper_NO_Small
- B1: footprint Button_Switch_THT:4-direction-joystick -> Button_Switch_THT:JS5208
- J4: value Conn_02x03_Odd_Even -> Conn_02x03
- SW1, SW2, SW3, SWPPT1: footprint Button_Switch_SMD:Panasonic_EVQPUM_EVQPUD -> Button_Switch_SMD:Reichelt_RAFI_Kurzhubtaster
- Y1: value Crystal -> 16MHz; footprint Crystal:Crystal_SMD_TXC_7A-2Pin_5x3.2mm -> Crystal:Crystal_SMD_5032-2Pin_5.0x3.2mm_HandSoldering
Connections:
- net +5V: now also C4.1, C5.1
- net D+: now also J1.2 (Pin_2)
- net D-: now also J1.1 (Pin_1)
- net GND: now also C4.2, C5.2, JP1.1
- net at J4.5 (Pin_5), U1.13 (~RESET): now also JP1.2
- net at U1.18 (PD0): now also B1.3 (PUSH); no longer SW1.1
- net at U1.19 (PD1): now also B1.2 (Left); no longer SW2.1
- net at U1.20 (PD2): now also B1.1 (Common); no longer SW3.1
- net at U1.22 (PD5): now also B1.4 (DOWN); no longer B1.1 (Common)
- net at U1.25 (PD4): now also SW1.1; no longer B1.4 (DOWN)
- net at U1.26 (PD6): now also SW2.1; no longer B1.2 (Left)
- net at U1.27 (PD7): now also SW3.1; no longer B1.3 (PUSH)
- no-connect marks 17 -> 16
Other:
- moved on the sheet: B1, J3, R2, R3, SW1, SW2, SW3, SWPPT1

Commit message: Add files via upload
Parts:
- added J2: Conn_01x02, Connector_PinHeader_2.54mm:PinHeader_1x02_P2.54mm_Vertical, symbol Connector_Generic:Conn_01x02
Connections:
- net +5V: now also J2.2 (Pin_2)
- net GND: now also J2.1 (Pin_1)
Changed lines of the file:
@@
 Text Label 4400 3250 0    50   ~ 0
 D+
+$Comp
+L Connector_Generic:Conn_01x02 J2
+U 1 1 5E36FB85
+P 3700 3100
+F 0 "J2" H 3700 3200 50  0000 C CNN
+F 1 "Conn_01x02" H 3700 3300 50  0000 C CNN
+F 2 "Connector_PinHeader_2.54mm:PinHeader_1x02_P2.54mm_Vertical" H 3700 3100 50  0001 C CNN
+F 3 "~" H 3700 3100 50  0001 C CNN
+	1    3700 3100
+	-1   0    0    1
+$EndComp
+$Comp
+L power:+5V #PWR02
+U 1 1 5E372F2D
+P 3900 3000
+F 0 "#PWR02" H 3900 2850 50  0001 C CNN
+F 1 "+5V" H 3915 3173 50  0000 C CNN
+F 2 "" H 3900 3000 50  0001 C CNN
+F 3 "" H 3900 3000 50  0001 C CNN
+	1    3900 3000
+	1    0    0    -1
+$EndComp
+$Comp
+L power:GND #PWR04
+U 1 1 5E37355B
+P 3900 3100
+F 0 "#PWR04" H 3900 2850 50  0001 C CNN
+F 1 "GND" H 3905 2927 50  0000 C CNN
+F 2 "" H 3900 3100 50  0001 C CNN
+F 3 "" H 3900 3100 50  0001 C CNN
+	1    3900 3100
+	1    0    0    -1
+$EndComp
 $EndSCHEMATC

Commit message: Add files via upload
Parts:
- added D2: LED, LED_SMD:LED_0805_2012Metric_Pad1.15x1.40mm_HandSolder, symbol Device:LED
- added F1: 500mA, Fuse:Fuse_0603_1608Metric, symbol Device:Fuse
- added R4: 1K, Resistor_SMD:R_0805_2012Metric_Pad1.15x1.40mm_HandSolder, symbol Device:R
Connections:
- net +5V: now also F1.1; no longer J2.2 (Pin_2)
- net GND: now also D2.1 (K)
- net at U1.1 (PE6): now also R4.2
- new net: F1.2, J2.2 (Pin_2)
- new net: D2.2 (A), R4.1
- no-connect marks 16 -> 15
Changed lines of the file:
@@
 	7750 1850 7500 1850
 Wire Wire Line
-	6650 3850 6650 4200
-Wire Wire Line
-	6650 4200 7400 4200
-Wire Wire Line
-	6550 4050 6550 4400
-Wire Wire Line
-	6550 4400 7400 4400
-Wire Wire Line
-	6450 4150 6450 4600
-Wire Wire Line
-	6450 4600 7400 4600
+	6800 3850 6800 4200
+Wire Wire Line
+	6800 4200 7400 4200
+Wire Wire Line
+	6700 4050 6700 4400
+Wire Wire Line
+	6700 4400 7400 4400
+Wire Wire Line
+	6600 4150 6600 4600
+Wire Wire Line
+	6600 4600 7400 4600
 Wire Wire Line
 	6450 3450 6450 3250
@@
 NoConn ~ 6350 2650
 Wire Wire Line
-	6350 4150 6450 4150
-Wire Wire Line
-	6350 4050 6550 4050
-Wire Wire Line
-	6350 3850 6650 3850
+	6350 4150 6600 4150
+Wire Wire Line
+	6350 4050 6700 4050
+Wire Wire Line
+	6350 3850 6800 3850
 Wire Wire Line
 	5850 1950 5850 1850
@@
 Wire Wire Line
 	6350 2450 7750 2450
-NoConn ~ 6350 4450
 $Comp
 L Device:R R2
@@
 L power:+5V #PWR02
 U 1 1 5E372F2D
-P 3900 3000
-F 0 "#PWR02" H 3900 2850 50  0001 C CNN
-F 1 "+5V" H 3915 3173 50  0000 C CNN
-F 2 "" H 3900 3000 50  0001 C CNN
-F 3 "" H 3900 3000 50  0001 C CNN
-	1    3900 3000
+P 3900 2650
+F 0 "#PWR02" H 3900 2500 50  0001 C CNN
+F 1 "+5V" H 3915 2823 50  0000 C CNN
+F 2 "" H 3900 2650 50  0001 C CNN
+F 3 "" H 3900 2650 50  0001 C CNN
+	1    3900 2650
 	1    0    0    -1
 $EndComp
@@
 	1    0    0    -1
 $EndComp
+$Comp
+L power:GND #PWR017
+U 1 1 5E37EFEA
+P 6500 5650
+F 0 "#PWR017" H 6500 5400 50  0001 C CNN
+F 1 "GND" H 6505 5477 50  0000 C CNN
+F 2 "" H 6500 5650 50  0001 C CNN
+F 3 "" H 6500 5650 50  0001 C CNN
+	1    6500 5650
+	1    0    0    -1
+$EndComp
+$Comp
+L Device:R R4
+U 1 1 5E37EFF0
+P 6500 5200
+F 0 "R4" V 6400 5200 50  0000 C CNN
+F 1 "1K" V 6500 5200 50  0000 C CNN
+F 2 "Resistor_SMD:R_0805_2012Metric_Pad1.15x1.40mm_HandSolder" V 6430 5200 50  0001 C CNN
+F 3 "~" H 6500 5200 50  0001 C CNN
+	1    6500 5200
+	-1   0    0    1
+$EndComp
+$Comp
+L Device:LED D2
+U 1 1 5E37EFF6
+P 6500 5500
+F 0 "D2" V 6539 5383 50  0000 R CNN
+F 1 "LED" V 6448 5383 50  0000 R CNN
+F 2 "LED_SMD:LED_0805_2012Metric_Pad1.15x1.40mm_HandSolder" H 6500 5500 50  0001 C CNN
+F 3 "~" H 6500 5500 50  0001 C CNN
+	1    6500 5500
+	0    -1   -1   0
+$EndComp
+Wire Wire Line
+	6350 4450 6500 4450
+Wire Wire Line
+	6500 4450 6500 5050
+$Comp
+L Device:Fuse F1
+U 1 1 5E3D934A
+P 3900 2800
+F 0 "F1" H 3960 2846 50  0000 L CNN
+F 1 "500mA" H 3960 2755 50  0000 L CNN
+F 2 "Fuse:Fuse_0603_1608Metric" V 3830 2800 50  0001 C CNN
+F 3 "~" H 3900 2800 50  0001 C CNN
+	1    3900 2800
+	1    0    0    -1
+$EndComp
+Wire Wire Line
+	3900 3000 3900 2950
 $EndSCHEMATC

Commit message: Add files via upload
Parts:
- added J5: Conn_01x02, Connector_Wire:SolderWirePadOval_2, symbol Connector_Generic:Conn_01x02
- J1, J2, J3: footprint Connector_PinHeader_2.54mm:PinHeader_1x02_P2.54mm_Vertical -> Connector_Wire:SolderWirePadOval_2
Connections:
- net GND: now also J5.2 (Pin_2)
- net at U1.12 (PB7): now also J5.1 (Pin_1)
- no-connect marks 15 -> 14
Other:
- moved on the sheet: C4, C5, D1, F1, J2, R1
Changed lines of the file:
@@
 L power:+5V #PWR06
 U 1 1 5E2D65E5
-P 4350 4200
-F 0 "#PWR06" H 4350 4050 50  0001 C CNN
-F 1 "+5V" H 4365 4373 50  0000 C CNN
-F 2 "" H 4350 4200 50  0001 C CNN
-F 3 "" H 4350 4200 50  0001 C CNN
-	1    4350 4200
+P 2750 3000
+F 0 "#PWR06" H 2750 2850 50  0001 C CNN
+F 1 "+5V" H 2765 3173 50  0000 C CNN
+F 2 "" H 2750 3000 50  0001 C CNN
+F 3 "" H 2750 3000 50  0001 C CNN
+	1    2750 3000
 	1    0    0    -1
 $EndComp
@@
 L power:GND #PWR07
 U 1 1 5E2D6D93
-P 4350 4800
-F 0 "#PWR07" H 4350 4550 50  0001 C CNN
-F 1 "GND" H 4355 4627 50  0000 C CNN
-F 2 "" H 4350 4800 50  0001 C CNN
-F 3 "" H 4350 4800 50  0001 C CNN
-	1    4350 4800
+P 2750 3600
+F 0 "#PWR07" H 2750 3350 50  0001 C CNN
+F 1 "GND" H 2755 3427 50  0000 C CNN
+F 2 "" H 2750 3600 50  0001 C CNN
+F 3 "" H 2750 3600 50  0001 C CNN
+	1    2750 3600
 	1    0    0    -1
 $EndComp
@@
 L Device:R R1
 U 1 1 5E2D762B
-P 4350 4350
-F 0 "R1" V 4250 4350 50  0000 C CNN
-F 1 "1K" V 4350 4350 50  0000 C CNN
-F 2 "Resistor_SMD:R_0805_2012Metric_Pad1.15x1.40mm_HandSolder" V 4280 4350 50  0001 C CNN
-F 3 "~" H 4350 4350 50  0001 C CNN
-	1    4350 4350
+P 2750 3150
+F 0 "R1" V 2650 3150 50  0000 C CNN
+F 1 "1K" V 2750 3150 50  0000 C CNN
+F 2 "Resistor_SMD:R_0805_2012Metric_Pad1.15x1.40mm_HandSolder" V 2680 3150 50  0001 C CNN
+F 3 "~" H 2750 3150 50  0001 C CNN
+	1    2750 3150
 	-1   0    0    1
 $EndComp
@@
 L Device:LED D1
 U 1 1 5E2D8127
-P 4350 4650
-F 0 "D1" V 4389 4533 50  0000 R CNN
-F 1 "LED" V 4298 4533 50  0000 R CNN
-F 2 "LED_SMD:LED_0805_2012Metric_Pad1.15x1.40mm_HandSolder" H 4350 4650 50  0001 C CNN
-F 3 "~" H 4350 4650 50  0001 C CNN
-	1    4350 4650
+P 2750 3450
+F 0 "D1" V 2789 3333 50  0000 R CNN
+F 1 "LED" V 2698 3333 50  0000 R CNN
+F 2 "LED_SMD:LED_0805_2012Metric_Pad1.15x1.40mm_HandSolder" H 2750 3450 50  0001 C CNN
+F 3 "~" H 2750 3450 50  0001 C CNN
+	1    2750 3450
 	0    -1   -1   0
 $EndComp
@@
 	1    0    0    -1
 $EndComp
-$Comp
-L Connector_Generic:Conn_01x02 J3
-U 1 1 5E312D11
-P 8300 5200
-F 0 "J3" H 8300 5300 50  0000 C CNN
-F 1 "Conn_01x02" H 8300 5400 50  0000 C CNN
-F 2 "Connector_PinHeader_2.54mm:PinHeader_1x02_P2.54mm_Vertical" H 8300 5200 50  0001 C CNN
-F 3 "~" H 8300 5200 50  0001 C CNN
-	1    8300 5200
-	1    0    0    -1
-$EndComp
 Wire Wire Line
 	7800 4700 7800 4600
@@
 L Device:C C4
 U 1 1 5E305386
-P 2750 2450
-F 0 "C4" H 2865 2496 50  0000 L CNN
-F 1 "0.1uF" H 2865 2405 50  0000 L CNN
-F 2 "Capacitor_SMD:C_0805_2012Metric_Pad1.15x1.40mm_HandSolder" H 2788 2300 50  0001 C CNN
-F 3 "~" H 2750 2450 50  0001 C CNN
-	1    2750 2450
+P 1150 3400
+F 0 "C4" H 1265 3446 50  0000 L CNN
+F 1 "0.1uF" H 1265 3355 50  0000 L CNN
+F 2 "Capacitor_SMD:C_0805_2012Metric_Pad1.15x1.40mm_HandSolder" H 1188 3250 50  0001 C CNN
+F 3 "~" H 1150 3400 50  0001 C CNN
+	1    1150 3400
 	1    0    0    -1
 $EndComp
@@
 L Device:C C5
 U 1 1 5E305E95
-P 3150 2450
-F 0 "C5" H 3265 2496 50  0000 L CNN
-F 1 "10uF" H 3265 2405 50  0000 L CNN
-F 2 "Capacitor_SMD:C_0805_2012Metric_Pad1.15x1.40mm_HandSolder" H 3188 2300 50  0001 C CNN
-F 3 "~" H 3150 2450 50  0001 C CNN
-	1    3150 2450
-	1    0    0    -1
-$EndComp
-Wire Wire Line
-	2750 2300 2950 2300
-Wire Wire Line
-	3150 2600 2950 2600
+P 1550 3400
+F 0 "C5" H 1665 3446 50  0000 L CNN
+F 1 "10uF" H 1665 3355 50  0000 L CNN
+F 2 "Capacitor_SMD:C_0805_2012Metric_Pad1.15x1.40mm_HandSolder" H 1588 3250 50  0001 C CNN
+F 3 "~" H 1550 3400 50  0001 C CNN
+	1    1550 3400
+	1    0    0    -1
+$EndComp
+Wire Wire Line
+	1150 3250 1350 3250
+Wire Wire Line
+	1550 3550 1350 3550
 $Comp
 L power:GND #PWR016
 U 1 1 5E30A54C
-P 2950 2600
-F 0 "#PWR016" H 2950 2350 50  0001 C CNN
-F 1 "GND" H 2955 2427 50  0000 C CNN
-F 2 "" H 2950 2600 50  0001 C CNN
-F 3 "" H 2950 2600 50  0001 C CNN
-	1    2950 2600
-	1    0    0    -1
-$EndComp
-Connection ~ 2950 2600
-Wire Wire Line
-	2950 2600 2750 2600
+P 1350 3550
+F 0 "#PWR016" H 1350 3300 50  0001 C CNN
+F 1 "GND" H 1355 3377 50  0000 C CNN
+F 2 "" H 1350 3550 50  0001 C CNN
+F 3 "" H 1350 3550 50  0001 C CNN
+	1    1350 3550
+	1    0    0    -1
+$EndComp
+Connection ~ 1350 3550
+Wire Wire Line
+	1350 3550 1150 3550
 $Comp
 L power:+5V #PWR03
 U 1 1 5E30AC51
-P 2950 2300
-F 0 "#PWR03" H 2950 2150 50  0001 C CNN
-F 1 "+5V" H 2965 2473 50  0000 C CNN
-F 2 "" H 2950 2300 50  0001 C CNN
-F 3 "" H 2950 2300 50  0001 C CNN
-	1    2950 2300
-	1    0    0    -1
-$EndComp
-Connection ~ 2950 2300
-Wire Wire Line
-	2950 2300 3150 2300
+P 1350 3250
+F 0 "#PWR03" H 1350 3100 50  0001 C CNN
+F 1 "+5V" H 1365 3423 50  0000 C CNN
+F 2 "" H 1350 3250 50  0001 C CNN
+F 3 "" H 1350 3250 50  0001 C CNN
+	1    1350 3250
+	1    0    0    -1
+$EndComp
+Connection ~ 1350 3250
+Wire Wire Line
+	1350 3250 1550 3250
 $Comp
 L Device:Jumper_NO_Small JP1
@@
 F 0 "J1" H 4200 3450 50  0000 C CNN
 F 1 "Conn_01x02" H 4200 3550 50  0000 C CNN
-F 2 "Connector_PinHeader_2.54mm:PinHeader_1x02_P2.54mm_Vertical" H 4200 3350 50  0001 C CNN
+F 2 "Connector_Wire:SolderWirePadOval_2" H 4200 3350 50  0001 C CNN
 F 3 "~" H 4200 3350 50  0001 C CNN
 	1    4200 3350
@@
 Wire Wire Line
 	5150 1950 5150 2250
-NoConn ~ 6350 2950
 Wire Wire Line
 	6350 2550 6700 2550
@@
 D+
 $Comp
-L Connector_Generic:Conn_01x02 J2
-U 1 1 5E36FB85
-P 3700 3100
-F 0 "J2" H 3700 3200 50  0000 C CNN
-F 1 "Conn_01x02" H 3700 3300 50  0000 C CNN
-F 2 "Connector_PinHeader_2.54mm:PinHeader_1x02_P2.54mm_Vertical" H 3700 3100 50  0001 C CNN
-F 3 "~" H 3700 3100 50  0001 C CNN
-	1    3700 3100
-	-1   0    0    1
-$EndComp
-$Comp
 L power:+5V #PWR02
 U 1 1 5E372F2D
-P 3900 2650
-F 0 "#PWR02" H 3900 2500 50  0001 C CNN
-F 1 "+5V" H 3915 2823 50  0000 C CNN
-F 2 "" H 3900 2650 50  0001 C CNN
-F 3 "" H 3900 2650 50  0001 C CNN
-	1    3900 2650
+P 2150 3000
+F 0 "#PWR02" H 2150 2850 50  0001 C CNN
+F 1 "+5V" H 2165 3173 50  0000 C CNN
+F 2 "" H 2150 3000 50  0001 C CNN
+F 3 "" H 2150 3000 50  0001 C CNN
+	1    2150 3000
 	1    0    0    -1
 $EndComp
@@
 L power:GND #PWR04
 U 1 1 5E37355B
-P 3900 3100
-F 0 "#PWR04" H 3900 2850 50  0001 C CNN
-F 1 "GND" H 3905 2927 50  0000 C CNN
-F 2 "" H 3900 3100 50  0001 C CNN
-F 3 "" H 3900 3100 50  0001 C CNN
-	1    3900 3100
+P 2150 3450
+F 0 "#PWR04" H 2150 3200 50  0001 C CNN
+F 1 "GND" H 2155 3277 50  0000 C CNN
+F 2 "" H 2150 3450 50  0001 C CNN
+F 3 "" H 2150 3450 50  0001 C CNN
+	1    2150 3450
 	1    0    0    -1
 $EndComp
@@
 L Device:Fuse F1
 U 1 1 5E3D934A
-P 3900 2800
-F 0 "F1" H 3960 2846 50  0000 L CNN
-F 1 "500mA" H 3960 2755 50  0000 L CNN
-F 2 "Fuse:Fuse_0603_1608Metric" V 3830 2800 50  0001 C CNN
-F 3 "~" H 3900 2800 50  0001 C CNN
-	1    3900 2800
-	1    0    0    -1
-$EndComp
-Wire Wire Line
-	3900 3000 3900 2950
+P 2150 3150
+F 0 "F1" H 2210 3196 50  0000 L CNN
+F 1 "500mA" H 2210 3105 50  0000 L CNN
+F 2 "Fuse:Fuse_0603_1608Metric" V 2080 3150 50  0001 C CNN
+F 3 "~" H 2150 3150 50  0001 C CNN
+	1    2150 3150
+	1    0    0    -1
+$EndComp
+Wire Wire Line
+	2150 3350 2150 3300
+Wire Wire Line
+	6350 2950 6900 2950
+Wire Wire Line
+	6900 2950 6900 2600
+Wire Wire Line
+	6900 2600 8050 2600
+Wire Wire Line
+	8050 2600 8050 2350
+Wire Wire Line
+	8050 2350 8300 2350
+$Comp
+L power:GND #PWR018
+U 1 1 5E4367F5
+P 8300 2600
+F 0 "#PWR018" H 8300 2350 50  0001 C CNN
+F 1 "GND" H 8305 2427 50  0000 C CNN
+F 2 "" H 8300 2600 50  0001 C CNN
+F 3 "" H 8300 2600 50  0001 C CNN
+	1    8300 2600
+	1    0    0    -1
+$EndComp
+Wire Wire Line
+	8300 2600 8300 2450
+$Comp
+L Connector_Generic:Conn_01x02 J3
+U 1 1 5E312D11
+P 8300 5200
+F 0 "J3" H 8300 5300 50  0000 C CNN
+F 1 "Conn_01x02" H 8300 5400 50  0000 C CNN
+F 2 "Connector_Wire:SolderWirePadOval_2" H 8300 5200 50  0001 C CNN
+F 3 "~" H 8300 5200 50  0001 C CNN
+	1    8300 5200
+	1    0    0    -1
+$EndComp
+$Comp
+L Connector_Generic:Conn_01x02 J2
+U 1 1 5E36FB85
+P 1950 3450
+F 0 "J2" H 1950 3550 50  0000 C CNN
+F 1 "Conn_01x02" H 1950 3650 50  0000 C CNN
+F 2 "Connector_Wire:SolderWirePadOval_2" H 1950 3450 50  0001 C CNN
+F 3 "~" H 1950 3450 50  0001 C CNN
+	1    1950 3450
+	-1   0    0    1
+$EndComp
+$Comp
+L Connector_Generic:Conn_01x02 J5
+U 1 1 5E431055
+P 8500 2350
+F 0 "J5" H 8500 2450 50  0000 C CNN
+F 1 "Conn_01x02" H 8500 2550 50  0000 C CNN
+F 2 "Connector_Wire:SolderWirePadOval_2" H 8500 2350 50  0001 C CNN
+F 3 "~" H 8500 2350 50  0001 C CNN
+	1    8500 2350
+	1    0    0    -1
+$EndComp
 $EndSCHEMATC
